File: KiCad/SpotWelder - Arduino Pro Mini vA/SpotWelder - Arduino Pro Mini vA.kicad_pcb (KiCad board)
At the start: 2 copper layers, 62.9 x 65.4 mm, 21 parts, among them U1 KY-040_Rotary_Encoder, U2 Switch, U3 Switch, U4 Arduino_Mini_Pro, U5 SSD1306_I2C_display, U6 SSR_Relay

Commit message: new sketches
Parts:
- U4: footprint My_Arduino:Arduino_Pro_Mini_vC_no-progr-large -> My_Arduino:Arduino_Pro_Mini_vA_sides_n_A4,A5_large
- moved U5 7.00 mm to (135.3, 118.6), turned to 90 degrees
Routing:
- net Net-(U4-A5): track 21.4 -> 35.3 mm
- net Net-(U4-A4): track 21.4 -> 28.4 mm
- net +5V: track 168.8 -> 163.8 mm
- net GND: track 178.1 -> 182.1 mm
