File: KiCad/SpotWelder - Arduino Pro Mini vA/SpotWelder - Arduino Pro Mini vA.kicad_sch (KiCad schematic)
At the start: 21 parts, among them U1 KY-040_Rotary_Encoder, U2 Switch, U3 Switch, U4 Arduino_Mini_Pro, U5 SSD1306_I2C_display, U6 SSR_Relay

Commit message: new sketches
Parts:
- U4: footprint My_Arduino:Arduino_Pro_Mini_vC_no-progr-large -> My_Arduino:Arduino_Pro_Mini_vA_sides_n_A4,A5_large
Changed lines of the file:
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@@
 			)
 		)
-		(property "Footprint" "My_Arduino:Arduino_Pro_Mini_vC_no-progr-large"
+		(property "Footprint" "My_Arduino:Arduino_Pro_Mini_vA_sides_n_A4,A5_large"
 			(at 181.61 92.71 0)
 			(effects
